File: KiCad/MicPreamp/MicPreamp.sch (KiCad schematic (older format))
At the start: 13 parts

Commit message: Mic preamp PCB done
Parts:
- added C2, C8: 10uf, Capacitors_SMD:C_0603, symbol Device:C
- added C3: 0.47uf, Capacitors_SMD:C_0603, symbol Device:C
- added R1: 100, Resistors_SMD:R_0603, symbol Device:R
- added R4: 50K, Resistors_SMD:R_0603, symbol Device:R
- added U2: LT3042, Housings_SSOP:MSOP-10-1EP_3x3mm_Pitch0.5mm, symbol IC_Generic:IC10
- C1, C7: renamed from C?; footprint (none) -> Capacitors_SMD:C_0603
- C4, C5, C6: renamed from C?; value 100n -> 1uf; footprint (none) -> Capacitors_SMD:C_0603
- J1, J3, J4, J5: renamed from J?; footprint (none) -> KiCadCustomLibs:Conn_1x02_2.54mm
- J2: renamed from J?; footprint (none) -> KiCadCustomLibs:Conn_1x01_2.54mm
- R2, R3: renamed from R?; footprint (none) -> Resistors_SMD:R_0603
- U1: renamed from U?; footprint (none) -> Housings_SSOP:TSSOP-10_3x3mm_Pitch0.5mm
Connections:
- net labels added: +9V
- wire segments 34 -> 56
- no-connect marks 0 -> 1
