File: KiCad/AudioProcessor/AudioProcessor.sch (KiCad schematic (older format))
At the start: 33 parts, among them J1 IN4, J2 IN3, J3 IN2, J4 IN1, J5 AUX, J6 I2C, J7 LOUT, J8 ROUT, J9 POWER, U1 TDA7440

Commit message: in progress
Parts:
- C13: value 2.2uf -> 10uf
Changed lines of the file:
@@
 EESchema Schematic File Version 4
+LIBS:AudioProcessor-cache
 EELAYER 26 0
 EELAYER END
@@
 P 7100 3250
 F 0 "C13" V 6950 3150 50  0000 L CNN
-F 1 "2.2uf" V 7250 3150 50  0000 L CNN
+F 1 "10uf" V 7250 3150 50  0000 L CNN
 F 2 "Capacitors_THT:C_Rect_L7.0mm_W2.0mm_P5.00mm" H 7138 3100 50  0001 C CNN
 F 3 "~" H 7100 3250 50  0001 C CNN

Commit message: Audio processor PCB is ready
Parts:
- removed C1, C3, C4: 2.2uf, Capacitors_THT:C_Rect_L7.0mm_W2.0mm_P5.00mm, symbol Device:C
- removed J5: AUX, Pin_Headers:Pin_Header_Straight_1x03_Pitch2.54mm, symbol Connector_Generic:Conn_01x03
- removed R4, R5, R6, R7, R8: 600, Resistors_SMD:R_0603, symbol Device:R
- added C1: 220uf, Capacitors_THT:CP_Radial_Tantal_D8.0mm_P5.00mm, symbol Device:CP1
- added C14, C15, C16, C17, C18, C19, C20, C21: 2uf, Capacitors_SMD:C_0603, symbol Device:C_Small
- added C22, C3: 100uf, Capacitors_THT:CP_Radial_Tantal_D6.0mm_P5.00mm, symbol Device:CP1
- added C23: 4.7n, Capacitors_THT:C_Rect_L7.0mm_W2.0mm_P5.00mm, symbol Device:C
- added C24: 1n, Capacitors_THT:C_Rect_L7.0mm_W2.0mm_P5.00mm, symbol Device:C
- added C4: 10uf, Capacitors_THT:CP_Radial_Tantal_D4.5mm_P2.50mm, symbol Device:CP1
- added J10: D_POT_PHONES, KiCadCustomLibs:Conn_1x03_2.54mm, symbol Connector_Generic:Conn_01x03
- added J5: PHONES, KiCadCustomLibs:Conn_1x02_2.54mm, symbol Connector_Generic:Conn_01x02
- added U2: LM386M, Housings_SOIC:SOIC-8_3.9x4.9mm_Pitch1.27mm, symbol Amplifier_Audio:LM386
- C11: value 5.6n -> 4.7n
- C12: value 5.6n -> 1n
- C13, C6, C7: footprint Capacitors_THT:C_Rect_L7.0mm_W2.0mm_P5.00mm -> Capacitors_SMD:C_0603
- C2: value 2.2uf -> 50n; footprint Capacitors_THT:C_Rect_L7.0mm_W2.0mm_P5.00mm -> Capacitors_SMD:C_0603
- J1, J2, J3, J4, J7, J8, J9: footprint KiCadCustomLibs:Conn2pin_2.54mm -> KiCadCustomLibs:Conn_1x02_2.54mm
- J6: footprint Pin_Headers:Pin_Header_Straight_1x03_Pitch2.54mm -> KiCadCustomLibs:Conn_1x03_2.54mm
- R1: value 600 -> 10
- R2, R3: value 600 -> 47K
Connections:
- net labels added: AUX
- wire segments 90 -> 125
- no-connect marks 2 -> 5

Commit message: Adjust components according to availability
Parts:
- C10, C5, C8, C9: footprint Capacitors_THT:C_Rect_L7.0mm_W2.0mm_P5.00mm -> Capacitors_THT:C_Rect_L7.2mm_W2.5mm_P5.00mm_FKS2_FKP2_MKS2_MKP2
- C11, C23: value 4.7n -> 5.6n; footprint Capacitors_THT:C_Rect_L7.0mm_W2.0mm_P5.00mm -> Capacitors_SMD:C_0805
- C12, C24: value 1n -> opt; footprint Capacitors_THT:C_Rect_L7.0mm_W2.0mm_P5.00mm -> Capacitors_SMD:C_0805
- U2: footprint Housings_SOIC:SOIC-8_3.9x4.9mm_Pitch1.27mm -> Housings_DIP:DIP-8_W7.62mm_Socket
Changed lines of the file:
@@
 P 8300 3700
 F 0 "C12" V 8250 3500 50  0000 L CNN
-F 1 "1n" V 8150 3600 50  0000 L CNN
-F 2 "Capacitors_THT:C_Rect_L7.0mm_W2.0mm_P5.00mm" H 8338 3550 50  0001 C CNN
+F 1 "opt" V 8150 3600 50  0000 L CNN
+F 2 "Capacitors_SMD:C_0805" H 8338 3550 50  0001 C CNN
 F 3 "~" H 8300 3700 50  0001 C CNN
 	1    8300 3700
@@
 F 0 "C9" V 7100 4050 50  0000 L CNN
 F 1 "100n" V 7100 4200 50  0000 L CNN
-F 2 "Capacitors_THT:C_Rect_L7.0mm_W2.0mm_P5.00mm" H 6988 4100 50  0001 C CNN
+F 2 "Capacitors_THT:C_Rect_L7.2mm_W2.5mm_P5.00mm_FKS2_FKP2_MKS2_MKP2" H 6988 4100 50  0001 C CNN
 F 3 "~" H 6950 4250 50  0001 C CNN
 	1    6950 4250
@@
 F 0 "C10" V 7500 4050 50  0000 L CNN
 F 1 "100n" V 7500 4200 50  0000 L CNN
-F 2 "Capacitors_THT:C_Rect_L7.0mm_W2.0mm_P5.00mm" H 7388 4100 50  0001 C CNN
+F 2 "Capacitors_THT:C_Rect_L7.2mm_W2.5mm_P5.00mm_FKS2_FKP2_MKS2_MKP2" H 7388 4100 50  0001 C CNN
 F 3 "~" H 7350 4250 50  0001 C CNN
 	1    7350 4250
@@
 P 8300 3400
 F 0 "C11" V 8250 3200 50  0000 L CNN
-F 1 "4.7n" V 8150 3300 50  0000 L CNN
-F 2 "Capacitors_THT:C_Rect_L7.0mm_W2.0mm_P5.00mm" H 8338 3250 50  0001 C CNN
+F 1 "5.6n" V 8150 3300 50  0000 L CNN
+F 2 "Capacitors_SMD:C_0805" H 8338 3250 50  0001 C CNN
 F 3 "~" H 8300 3400 50  0001 C CNN
 	1    8300 3400
@@
 F 0 "C5" V 6300 4050 50  0000 L CNN
 F 1 "100n" V 6300 4200 50  0000 L CNN
-F 2 "Capacitors_THT:C_Rect_L7.0mm_W2.0mm_P5.00mm" H 6188 4100 50  0001 C CNN
+F 2 "Capacitors_THT:C_Rect_L7.2mm_W2.5mm_P5.00mm_FKS2_FKP2_MKS2_MKP2" H 6188 4100 50  0001 C CNN
 F 3 "~" H 6150 4250 50  0001 C CNN
 	1    6150 4250
@@
 F 0 "C8" V 6700 4050 50  0000 L CNN
 F 1 "100n" V 6700 4200 50  0000 L CNN
-F 2 "Capacitors_THT:C_Rect_L7.0mm_W2.0mm_P5.00mm" H 6588 4100 50  0001 C CNN
+F 2 "Capacitors_THT:C_Rect_L7.2mm_W2.5mm_P5.00mm_FKS2_FKP2_MKS2_MKP2" H 6588 4100 50  0001 C CNN
 F 3 "~" H 6550 4250 50  0001 C CNN
 	1    6550 4250
@@
 F 0 "U2" H 4150 3650 50  0000 L CNN
 F 1 "LM386M" H 4050 3900 50  0000 L CNN
-F 2 "Housings_SOIC:SOIC-8_3.9x4.9mm_Pitch1.27mm" H 4050 3850 50  0001 C CNN
+F 2 "Housings_DIP:DIP-8_W7.62mm_Socket" H 4050 3850 50  0001 C CNN
 F 3 "http://www.ti.com/lit/ds/symlink/lm386.pdf" H 4150 3950 50  0001 C CNN
 	1    3950 3750
@@
 P 8300 4300
 F 0 "C24" V 8250 4100 50  0000 L CNN
-F 1 "1n" V 8150 4200 50  0000 L CNN
-F 2 "Capacitors_THT:C_Rect_L7.0mm_W2.0mm_P5.00mm" H 8338 4150 50  0001 C CNN
+F 1 "opt" V 8150 4200 50  0000 L CNN
+F 2 "Capacitors_SMD:C_0805" H 8338 4150 50  0001 C CNN
 F 3 "~" H 8300 4300 50  0001 C CNN
 	1    8300 4300
@@
 P 8300 4000
 F 0 "C23" V 8250 3800 50  0000 L CNN
-F 1 "4.7n" V 8150 3900 50  0000 L CNN
-F 2 "Capacitors_THT:C_Rect_L7.0mm_W2.0mm_P5.00mm" H 8338 3850 50  0001 C CNN
+F 1 "5.6n" V 8150 3900 50  0000 L CNN
+F 2 "Capacitors_SMD:C_0805" H 8338 3850 50  0001 C CNN
 F 3 "~" H 8300 4000 50  0001 C CNN
 	1    8300 4000
