File: KiCad/Arduino/Arduino.sch (KiCad schematic (older format))
At the start: 18 parts

Commit message: Finished Arduino board
Parts:
- added C7, C8: 10uf, Capacitors_SMD:C_0603, symbol Device:C_Small
- added J13: D_Pots, KiCadCustomLibs:Conn_1x03_2.54mm, symbol Connector_Generic:Conn_01x03
- added J15: IN1_SENS, KiCadCustomLibs:Conn_1x01_2.54mm, symbol Connector_Generic:Conn_01x01
- added J16: 5V, KiCadCustomLibs:Conn_1x02_2.54mm, symbol Connector_Generic:Conn_01x02
- added J4: D10, KiCadCustomLibs:Conn_1x01_2.54mm, symbol Connector_Generic:Conn_01x01
- added J5: A3, KiCadCustomLibs:Conn_1x01_2.54mm, symbol Connector_Generic:Conn_01x01
- added J6: A2, KiCadCustomLibs:Conn_1x01_2.54mm, symbol Connector_Generic:Conn_01x01
- added J7: A1, KiCadCustomLibs:Conn_1x01_2.54mm, symbol Connector_Generic:Conn_01x01
- added J8: A0, KiCadCustomLibs:Conn_1x01_2.54mm, symbol Connector_Generic:Conn_01x01
- added J9: SPI, KiCadCustomLibs:Conn_1x04_2.54mm, symbol Connector_Generic:Conn_01x04
- added R5: 470, Resistors_SMD:R_0603, symbol Device:R_Small
- J14: renamed from J?; footprint KiCadCustomLibs:Conn2pin_2.54mm -> KiCadCustomLibs:Conn_1x02_2.54mm
- gave numbers to parts that had none: 17
Connections:
- net labels added: E0A, E0B, E0C, E1A, E1B, E1C, MISO, MOSI, SCK
- wire segments 66 -> 93
- no-connect marks 4 -> 6

Commit message: Digital pots board ready
Connections:
- net labels added: E0S, E1S
- net labels removed: E0C, E1C
Changed lines of the file:
@@
 E0B
 Text Label 3800 3650 0    50   ~ 0
-E0C
+E0S
 Text Label 3800 4200 0    50   ~ 0
 E1A
@@
 E1B
 Text Label 3800 4400 0    50   ~ 0
-E1C
+E1S
 $Comp
 L Connector_Generic:Conn_01x02 J16
