File: KiCad/Combined/Combined.kicad_pcb (KiCad board)
At the start: 2 copper layers, 91 x 79 mm, 120 parts, among them J1 Conn_01x04, J1 Enc_MAIN, J1 IN4, J1 PWR, J1 i2c, J10 D_POT, J10 VBAT, J11 Audio, J12 LCD, J13 D_Pots, J14 PWR, J15 IN1_SENS, J16 5V, J2 3, J2 Enc_INPUT, J2 IN3, J2 INT, J3 1, J3 IN2, J3 LED, J3 OUT, J4 2, J4 AUX, J4 D10, J4 IN1, J5 0, J5 A3, J5 MIC, J5 PHONES, J6 A2, J6 Conn_01x02, J6 I2C, J7 A1, J7 LOUT, J7 PWR, J8 A0, J8 ROUT, J9 POWER, J9 SPI, SW1 Rotary_Encoder_Switch, U1 LP2985-5.0, U1 MAX4062, U1 TDA7440, U2 IC20, U2 LM386M, U2 LT3042

Commit message: PCB's finished and sent to JLPCB
Parts:
- removed the J1 at (125.7, 81.0)
- removed the REF** at (118.8, 90.2)
- removed the REF** at (140.8, 90.2)
- added D1: WS2812B, LED_SMD:LED_WS2812B_PLCC4_5.0x5.0mm_P3.2mm, F.Cu at (144.0, 40.0)
- added D1: WS2812B, LED_SMD:LED_WS2812B_PLCC4_5.0x5.0mm_P3.2mm, F.Cu at (108.0, 40.0)
- added D1: WS2812B, LED_SMD:LED_WS2812B_PLCC4_5.0x5.0mm_P3.2mm, F.Cu at (90.0, 40.0)
- added D1: WS2812B, LED_SMD:LED_WS2812B_PLCC4_5.0x5.0mm_P3.2mm, F.Cu at (72.0, 40.0)
- added D1: WS2812B, LED_SMD:LED_WS2812B_PLCC4_5.0x5.0mm_P3.2mm, F.Cu at (148.5, 75.5)
- added D1: WS2812B, LED_SMD:LED_WS2812B_PLCC4_5.0x5.0mm_P3.2mm, F.Cu at (148.5, 94.5)
- added D2: WS2812B, LED_SMD:LED_WS2812B_PLCC4_5.0x5.0mm_P3.2mm, F.Cu at (138.0, 40.0)
- added D2: WS2812B, LED_SMD:LED_WS2812B_PLCC4_5.0x5.0mm_P3.2mm, F.Cu at (148.5, 69.5)
- added D3: WS2812B, LED_SMD:LED_WS2812B_PLCC4_5.0x5.0mm_P3.2mm, F.Cu at (132.1, 40.0)
- added D3: WS2812B, LED_SMD:LED_WS2812B_PLCC4_5.0x5.0mm_P3.2mm, F.Cu at (148.5, 63.6)
- added D4: WS2812B, LED_SMD:LED_WS2812B_PLCC4_5.0x5.0mm_P3.2mm, F.Cu at (126.0, 40.0)
- added D4: WS2812B, LED_SMD:LED_WS2812B_PLCC4_5.0x5.0mm_P3.2mm, F.Cu at (148.5, 57.5)
- added J1: IN, Connector_PinHeader_2.54mm:PinHeader_1x03_P2.54mm_Vertical, F.Cu at (150.0, 42.5)
- added J1: IN, Connector_PinHeader_2.54mm:PinHeader_1x03_P2.54mm_Vertical, F.Cu at (146.0, 100.5)
- added J1: IN, Connector_PinHeader_2.54mm:PinHeader_1x03_P2.54mm_Vertical, F.Cu at (114.0, 42.5)
- added J1: IN, Connector_PinHeader_2.54mm:PinHeader_1x03_P2.54mm_Vertical, F.Cu at (96.0, 42.5)
- added J1: IN, Connector_PinHeader_2.54mm:PinHeader_1x03_P2.54mm_Vertical, F.Cu at (78.0, 42.5)
- added J1: IN, Connector_PinHeader_2.54mm:PinHeader_1x03_P2.54mm_Vertical, F.Cu at (146.0, 81.5)
- added J1: Conn_01x04, KiCadCustomLibs:Conn_1x04_2.54mm, F.Cu at (120.5, 91.3)
- added J2: OUT, Connector_PinHeader_2.54mm:PinHeader_1x03_P2.54mm_Vertical, F.Cu at (120.0, 42.5)
- added J2: OUT, Connector_PinHeader_2.54mm:PinHeader_1x03_P2.54mm_Vertical, F.Cu at (146.0, 88.5)
- added J2: OUT, Connector_PinHeader_2.54mm:PinHeader_1x03_P2.54mm_Vertical, F.Cu at (102.0, 42.5)
- added J2: OUT, Connector_PinHeader_2.54mm:PinHeader_1x03_P2.54mm_Vertical, F.Cu at (84.0, 42.5)
- added J2: OUT, Connector_PinHeader_2.54mm:PinHeader_1x03_P2.54mm_Vertical, F.Cu at (66.0, 42.5)
- added J2: OUT, Connector_PinHeader_2.54mm:PinHeader_1x03_P2.54mm_Vertical, F.Cu at (146.0, 51.5)
- added REF**: hole, KiCadCustomLibs:hole_0.7, F.Cu at (66.5, 46.5)
- added REF**: hole, KiCadCustomLibs:hole_0.7, F.Cu at (147.5, 44.5)
- added REF**: hole, KiCadCustomLibs:hole_0.7, F.Cu at (98.0, 84.5)
- added REF**: hole, KiCadCustomLibs:hole_0.7, F.Cu at (96.5, 84.5)
- added REF**: hole, KiCadCustomLibs:hole_0.7, F.Cu at (96.5, 82.5)
- added REF**: hole, KiCadCustomLibs:hole_0.7, F.Cu at (73.5, 84.5)
- added REF**: hole, KiCadCustomLibs:hole_0.7, F.Cu at (73.5, 82.5)
- added REF**: hole, KiCadCustomLibs:hole_0.7, F.Cu at (70.5, 84.5)
- added REF**: hole, KiCadCustomLibs:hole_0.7, F.Cu at (72.0, 84.5)
- added REF**: hole, KiCadCustomLibs:hole_0.7, F.Cu at (72.0, 82.5)
- added REF**: hole, KiCadCustomLibs:hole_0.7, F.Cu at (70.5, 82.5)
- added REF**: hole, KiCadCustomLibs:hole_0.7, F.Cu at (146.0, 44.5)
- added REF**: MountingHole_3mm, Mounting_Holes:MountingHole_3mm, F.Cu at (129.8, 98.2)
- added REF**: MountingHole_3mm, Mounting_Holes:MountingHole_3mm, F.Cu at (129.8, 76.2)
- added REF**: hole, KiCadCustomLibs:hole_0.7, F.Cu at (149.0, 44.5)
- added REF**: hole, KiCadCustomLibs:hole_0.7, F.Cu at (146.0, 49.5)
- added REF**: hole, KiCadCustomLibs:hole_0.7, F.Cu at (147.5, 49.5)
- added REF**: hole, KiCadCustomLibs:hole_0.7, F.Cu at (149.0, 49.5)
- added REF**: hole, KiCadCustomLibs:hole_0.7, F.Cu at (118.0, 41.5)
- added REF**: hole, KiCadCustomLibs:hole_0.7, F.Cu at (118.0, 38.5)
- added REF**: hole, KiCadCustomLibs:hole_0.7, F.Cu at (118.0, 40.0)
- added REF**: hole, KiCadCustomLibs:hole_0.7, F.Cu at (126.5, 44.5)
- added REF**: hole, KiCadCustomLibs:hole_0.7, F.Cu at (68.0, 46.5)
- added REF**: hole, KiCadCustomLibs:hole_0.7, F.Cu at (128.0, 44.5)
- added REF**: hole, KiCadCustomLibs:hole_0.7, F.Cu at (129.5, 44.5)
- added REF**: hole, KiCadCustomLibs:hole_0.7, F.Cu at (105.5, 44.5)
- added REF**: hole, KiCadCustomLibs:hole_0.7, F.Cu at (116.0, 40.0)
- added REF**: hole, KiCadCustomLibs:hole_0.7, F.Cu at (100.0, 38.5)
- added REF**: hole, KiCadCustomLibs:hole_0.7, F.Cu at (116.0, 41.5)
- added REF**: hole, KiCadCustomLibs:hole_0.7, F.Cu at (116.0, 38.5)
- added REF**: hole, KiCadCustomLibs:hole_0.7, F.Cu at (102.5, 44.5)
- added REF**: hole, KiCadCustomLibs:hole_0.7, F.Cu at (104.0, 44.5)
- added REF**: hole, KiCadCustomLibs:hole_0.7, F.Cu at (100.0, 40.0)
- added REF**: hole, KiCadCustomLibs:hole_0.7, F.Cu at (69.5, 46.5)
- added REF**: hole, KiCadCustomLibs:hole_0.7, F.Cu at (100.0, 41.5)
- added REF**: hole, KiCadCustomLibs:hole_0.7, F.Cu at (98.0, 41.5)
- added REF**: hole, KiCadCustomLibs:hole_0.7, F.Cu at (87.5, 44.5)
- added REF**: hole, KiCadCustomLibs:hole_0.7, F.Cu at (84.5, 44.5)
- added REF**: hole, KiCadCustomLibs:hole_0.7, F.Cu at (98.0, 38.5)
- added REF**: hole, KiCadCustomLibs:hole_0.7, F.Cu at (82.0, 38.5)
- added REF**: hole, KiCadCustomLibs:hole_0.7, F.Cu at (82.0, 40.0)
- added REF**: hole, KiCadCustomLibs:hole_0.7, F.Cu at (86.0, 44.5)
- added REF**: hole, KiCadCustomLibs:hole_0.7, F.Cu at (98.0, 40.0)
- added REF**: hole, KiCadCustomLibs:hole_0.7, F.Cu at (82.0, 41.5)
- added REF**: hole, KiCadCustomLibs:hole_0.7, F.Cu at (86.0, 46.5)
- added REF**: hole, KiCadCustomLibs:hole_0.7, F.Cu at (68.0, 44.5)
- added REF**: hole, KiCadCustomLibs:hole_0.7, F.Cu at (129.5, 49.5)
- added REF**: hole, KiCadCustomLibs:hole_0.7, F.Cu at (126.5, 49.5)
- added REF**: hole, KiCadCustomLibs:hole_0.7, F.Cu at (69.5, 44.5)
- added REF**: hole, KiCadCustomLibs:hole_0.7, F.Cu at (66.5, 44.5)
- added REF**: hole, KiCadCustomLibs:hole_0.7, F.Cu at (128.0, 49.5)
- added REF**: hole, KiCadCustomLibs:hole_0.7, F.Cu at (80.0, 41.5)
- added REF**: hole, KiCadCustomLibs:hole_0.7, F.Cu at (80.0, 38.5)
- added REF**: hole, KiCadCustomLibs:hole_0.7, F.Cu at (80.0, 40.0)
- added REF**: hole, KiCadCustomLibs:hole_0.7, F.Cu at (117.5, 64.5)
- added REF**: hole, KiCadCustomLibs:hole_0.7, F.Cu at (87.5, 46.5)
- added REF**: hole, KiCadCustomLibs:hole_0.7, F.Cu at (117.5, 66.0)
- added REF**: hole, KiCadCustomLibs:hole_0.7, F.Cu at (117.5, 67.5)
- added REF**: hole, KiCadCustomLibs:hole_0.7, F.Cu at (117.5, 52.5)
- added REF**: hole, KiCadCustomLibs:hole_0.7, F.Cu at (117.5, 54.0)
- added REF**: hole, KiCadCustomLibs:hole_0.7, F.Cu at (117.5, 55.5)
- added REF**: hole, KiCadCustomLibs:hole_0.7, F.Cu at (141.5, 61.0)
- added REF**: hole, KiCadCustomLibs:hole_0.7, F.Cu at (141.5, 59.5)
- added REF**: hole, KiCadCustomLibs:hole_0.7, F.Cu at (141.5, 58.0)
- added REF**: hole, KiCadCustomLibs:hole_0.7, F.Cu at (144.0, 92.0)
- added REF**: hole, KiCadCustomLibs:hole_0.7, F.Cu at (144.0, 89.0)
- added REF**: hole, KiCadCustomLibs:hole_0.7, F.Cu at (84.5, 46.5)
- added REF**: hole, KiCadCustomLibs:hole_0.7, F.Cu at (144.0, 90.5)
- added REF**: hole, KiCadCustomLibs:hole_0.7, F.Cu at (147.0, 83.5)
- added REF**: hole, KiCadCustomLibs:hole_0.7, F.Cu at (150.0, 83.5)
- added REF**: hole, KiCadCustomLibs:hole_0.7, F.Cu at (148.5, 83.5)
- added REF**: hole, KiCadCustomLibs:hole_0.7, F.Cu at (147.0, 86.5)
- added REF**: hole, KiCadCustomLibs:hole_0.7, F.Cu at (150.0, 86.5)
- added REF**: hole, KiCadCustomLibs:hole_0.7, F.Cu at (148.5, 86.5)
- added REF**: hole, KiCadCustomLibs:hole_0.7, F.Cu at (112.5, 92.0)
- added REF**: hole, KiCadCustomLibs:hole_0.7, F.Cu at (112.5, 89.0)
- added REF**: hole, KiCadCustomLibs:hole_0.7, F.Cu at (112.5, 90.5)
- added REF**: hole, KiCadCustomLibs:hole_0.7, F.Cu at (102.5, 46.5)
- added REF**: hole, KiCadCustomLibs:hole_0.7, F.Cu at (144.0, 61.0)
- added REF**: hole, KiCadCustomLibs:hole_0.7, F.Cu at (144.0, 59.5)
- added REF**: hole, KiCadCustomLibs:hole_0.7, F.Cu at (144.0, 58.0)
- added REF**: hole, KiCadCustomLibs:hole_0.7, F.Cu at (148.5, 102.5)
- added REF**: hole, KiCadCustomLibs:hole_0.7, F.Cu at (150.0, 102.5)
- added REF**: hole, KiCadCustomLibs:hole_0.7, F.Cu at (147.0, 102.5)
- added REF**: hole, KiCadCustomLibs:hole_0.7, F.Cu at (115.5, 67.5)
- added REF**: hole, KiCadCustomLibs:hole_0.7, F.Cu at (115.5, 64.5)
- added REF**: hole, KiCadCustomLibs:hole_0.7, F.Cu at (115.5, 66.0)
- added REF**: hole, KiCadCustomLibs:hole_0.7, F.Cu at (115.5, 54.0)
- added REF**: hole, KiCadCustomLibs:hole_0.7, F.Cu at (105.5, 46.5)
- added REF**: hole, KiCadCustomLibs:hole_0.7, F.Cu at (115.5, 52.5)
- added REF**: hole, KiCadCustomLibs:hole_0.7, F.Cu at (115.5, 55.5)
- added REF**: hole, KiCadCustomLibs:hole_0.7, F.Cu at (142.0, 90.5)
- added REF**: hole, KiCadCustomLibs:hole_0.7, F.Cu at (117.5, 90.5)
- added REF**: hole, KiCadCustomLibs:hole_0.7, F.Cu at (142.0, 89.0)
- added REF**: hole, KiCadCustomLibs:hole_0.7, F.Cu at (117.5, 92.0)
- added REF**: hole, KiCadCustomLibs:hole_0.7, F.Cu at (142.0, 92.0)
- added REF**: hole, KiCadCustomLibs:hole_0.7, F.Cu at (117.5, 89.0)
- added REF**: hole, KiCadCustomLibs:hole_0.7, F.Cu at (112.5, 110.5)
- added REF**: hole, KiCadCustomLibs:hole_0.7, F.Cu at (114.5, 110.5)
- added REF**: hole, KiCadCustomLibs:hole_0.7, F.Cu at (104.0, 46.5)
- added REF**: hole, KiCadCustomLibs:hole_0.7, F.Cu at (112.5, 109.0)
- added REF**: hole, KiCadCustomLibs:hole_0.7, F.Cu at (114.5, 112.0)
- added REF**: hole, KiCadCustomLibs:hole_0.7, F.Cu at (112.5, 112.0)
- added REF**: hole, KiCadCustomLibs:hole_0.7, F.Cu at (114.5, 109.0)
- added REF**: hole, KiCadCustomLibs:hole_0.7, F.Cu at (147.0, 104.5)
- added REF**: hole, KiCadCustomLibs:hole_0.7, F.Cu at (150.0, 104.5)
- added REF**: hole, KiCadCustomLibs:hole_0.7, F.Cu at (148.5, 104.5)
- added REF**: hole, KiCadCustomLibs:hole_0.7, F.Cu at (99.5, 82.5)
- added REF**: hole, KiCadCustomLibs:hole_0.7, F.Cu at (99.5, 84.5)
- added REF**: hole, KiCadCustomLibs:hole_0.7, F.Cu at (98.0, 82.5)
- moved J2 18.4 mm to (138.5, 66.9), turned to 180 degrees
- moved J1 15.3 mm to (138.5, 52.8), turned to 0 degrees
- moved J4 14.9 mm to (120.5, 64.2), turned to 0 degrees
- moved R1 14.6 mm to (133.3, 67.4), turned to 0 degrees
- moved J3 13.6 mm to (138.5, 59.7), turned to 0 degrees
- moved R3 13.4 mm to (130.1, 67.4), turned to 0 degrees
- moved J5 12.6 mm to (120.5, 60.7), turned to 180 degrees
- moved C4 11.7 mm to (125.0, 65.3), turned to 0 degrees
- moved C1 10.7 mm to (135.7, 87.3), turned to 270 degrees
- moved C8 9.71 mm to (123.9, 53.4), turned to 90 degrees
- moved U1 9.53 mm to (131.1, 64.4), turned to 180 degrees
- moved C5 9.23 mm to (125.0, 63.2), turned to 0 degrees
- moved C3 8.27 mm to (127.5, 52.4), turned to 90 degrees
- moved R4 7.96 mm to (129.6, 52.4), turned to 270 degrees
- moved R2 7.79 mm to (133.8, 60.7), turned to 90 degrees
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Routing:
- net Net-(D1-Pad1): track 0.00 -> 236.2 mm, vias 0 -> 12
- net Net-(D1-Pad3): track 0.00 -> 235.5 mm, vias 0 -> 12
- net Net-(D1-Pad4): track 0.00 -> 38.4 mm
- net Net-(D1-Pad2): track 0.00 -> 37.3 mm
- net Net-(D3-Pad2): track 0.00 -> 12.2 mm
- net Net-(D4-Pad2): track 0.00 -> 12.1 mm
- net Net-(D2-Pad2): track 0.00 -> 12.1 mm
Other:
- board size 91 x 79 mm -> 91.5 x 90 mm
- net class Default: clearance 0.3 -> 0.2; trace_width 0.5 -> 0.4; via_dia 1.2 -> 1; via_drill 0.6 -> 0.5
- net class PWR removed
- rule pad_to_mask_clearance: 0.1 -> 0.051
- rule trace_clearance: 0.3 -> 0.2

Commit message: various work
Parts:
- removed ARDUINO1: ARDUINO_NANO, KiCadCustomLibs:arduino_nano
- removed C1, C2 (x2), C3, C4, C5, C6: 10n, Capacitors_SMD:C_0603
- removed C1, C14, C15, C16, C17, C18, C19, C20, C21, C6, C7: 2uf, Capacitors_SMD:C_0603
- removed C1, C4, C7: 100n, Capacitors_SMD:C_0603
- removed C1, C2, C3: C_Small, Capacitors_SMD:C_0603
- removed C1: 220uf, Capacitors_THT:CP_Radial_Tantal_D8.0mm_P5.00mm
- removed C10, C5, C8, C9: 100n, Capacitors_THT:C_Rect_L7.2mm_W2.5mm_P5.00mm_FKS2_FKP2_MKS2_MKP2
- removed C11, C23: 4.7n, Capacitors_SMD:C_0805
- removed C12, C24: 1n, Capacitors_SMD:C_0805
- removed C13, C2, C3, C7, C8 (x2): 10uf, Capacitors_SMD:C_0603
- removed C2: 50n, Capacitors_SMD:C_0603
- removed C22, C3: 100uf, Capacitors_THT:CP_Radial_Tantal_D6.0mm_P5.00mm
- removed C3: 0.47uf, Capacitors_SMD:C_0603
- removed C4, C5, C6: 1uf, Capacitors_SMD:C_0603
- removed C4: 10uf, Capacitors_THT:CP_Radial_Tantal_D4.5mm_P2.50mm
- removed D1 (x6), D2 (x2), D3 (x2), D4 (x2): WS2812B, LED_SMD:LED_WS2812B_PLCC4_5.0x5.0mm_P3.2mm
- removed J1 (x6): IN, Connector_PinHeader_2.54mm:PinHeader_1x03_P2.54mm_Vertical
- removed J1: IN4, KiCadCustomLibs:Conn_1x02_2.54mm
- removed J1: Enc_MAIN, KiCadCustomLibs:Conn_1x04_2.54mm
- removed J1: i2c, KiCadCustomLibs:Conn_1x03_2.54mm
- removed J1, J14, J7: PWR, KiCadCustomLibs:Conn_1x02_2.54mm
- removed J1: Conn_01x04, KiCadCustomLibs:Conn_1x04_2.54mm
- removed J10: VBAT, KiCadCustomLibs:Conn_1x01_2.54mm
- removed J10: D_POT, KiCadCustomLibs:Conn_1x03_2.54mm
- removed J11: Audio, KiCadCustomLibs:Conn_1x03_2.54mm
- removed J12: LCD, KiCadCustomLibs:Conn_1x04_2.54mm
- removed J13: D_Pots, KiCadCustomLibs:Conn_1x03_2.54mm
- removed J15: IN1_SENS, KiCadCustomLibs:Conn_1x01_2.54mm
- removed J16: 5V, KiCadCustomLibs:Conn_1x02_2.54mm
- removed J2 (x6): OUT, Connector_PinHeader_2.54mm:PinHeader_1x03_P2.54mm_Vertical
- removed J2: Enc_INPUT, KiCadCustomLibs:Conn_1x04_2.54mm
- removed J2: 3, KiCadCustomLibs:Conn_1x03_2.54mm
- removed J2: INT, KiCadCustomLibs:Conn_1x01_2.54mm
- removed J2: IN3, KiCadCustomLibs:Conn_1x02_2.54mm
- removed J3: LED, KiCadCustomLibs:Conn_1x03_2.54mm
- removed J3: 1, KiCadCustomLibs:Conn_1x03_2.54mm
- removed J3: OUT, KiCadCustomLibs:Conn_1x02_2.54mm
- removed J3: IN2, KiCadCustomLibs:Conn_1x02_2.54mm
- removed J4: D10, KiCadCustomLibs:Conn_1x01_2.54mm
- removed J4: 2, KiCadCustomLibs:Conn_1x03_2.54mm
- removed J4: AUX, KiCadCustomLibs:Conn_1x02_2.54mm
- removed J4: IN1, KiCadCustomLibs:Conn_1x02_2.54mm
- removed J5: A3, KiCadCustomLibs:Conn_1x01_2.54mm
- removed J5: 0, KiCadCustomLibs:Conn_1x03_2.54mm
- removed J5: MIC, KiCadCustomLibs:Conn_1x02_2.54mm
- removed J5: PHONES, KiCadCustomLibs:Conn_1x02_2.54mm
- removed J6: A2, KiCadCustomLibs:Conn_1x01_2.54mm
- removed J6: Conn_01x02, KiCadCustomLibs:Conn_1x02_2.54mm
- removed J6: I2C, KiCadCustomLibs:Conn_1x03_2.54mm
- removed J7: A1, KiCadCustomLibs:Conn_1x01_2.54mm
- removed J7: LOUT, KiCadCustomLibs:Conn_1x02_2.54mm
- removed J8: A0, KiCadCustomLibs:Conn_1x01_2.54mm
- removed J8: ROUT, KiCadCustomLibs:Conn_1x02_2.54mm
- removed J9: SPI, KiCadCustomLibs:Conn_1x04_2.54mm
- removed J9: POWER, KiCadCustomLibs:Conn_1x02_2.54mm
- removed JP1: A0, Jumper:SolderJumper-3_P1.3mm_Open_Pad1.0x1.5mm_NumberLabels
- removed JP2: A1, Jumper:SolderJumper-3_P1.3mm_Open_Pad1.0x1.5mm_NumberLabels
- removed JP3: WP, Jumper:SolderJumper-3_P1.3mm_Open_Pad1.0x1.5mm_NumberLabels
- removed R1, R2: 3K, Resistors_SMD:R_0603
- removed R1: 10k, Resistors_SMD:R_0603
- removed R1: 100, Resistors_SMD:R_0603
- removed R1: 10, Resistors_SMD:R_0603
- removed R10, R9: 5.6k, Resistors_SMD:R_0603
- removed R2, R4: 100K, Resistors_SMD:R_0603
- removed R2, R3: 47K, Resistors_SMD:R_0603
- removed R3: 510K, Resistors_SMD:R_0603
- removed R3: 11K, Resistors_SMD:R_0603
- removed R4: 50K, Resistors_SMD:R_0603
- removed R5: 470, Resistors_SMD:R_0603
- removed REF** (x108): hole, KiCadCustomLibs:hole_0.7
- removed REF** (x8): MountingHole_3mm, Mounting_Holes:MountingHole_3mm
- removed SW1: Rotary_Encoder_Switch, KiCadCustomLibs:ROTARY-ENCODER
- removed U1: LP2985-5.0, TO_SOT_Packages_SMD:SOT-23-5
- removed U1: MAX4062, Housings_SSOP:TSSOP-10_3x3mm_Pitch0.5mm
- removed U1: TDA7440, Housings_SOIC:SOIC-28W_7.5x17.9mm_Pitch1.27mm
- removed U2: IC20, Housings_SSOP:TSSOP-20_4.4x6.5mm_Pitch0.65mm
- removed U2: LT3042, Housings_SSOP:MSOP-10-1EP_3x3mm_Pitch0.5mm
- removed U2: LM386M, Housings_DIP:DIP-8_W7.62mm_Socket
Routing:
- net Net-(D1-Pad1): track 236.2 -> 0.00 mm, vias 12 -> 0
- net Net-(D1-Pad3): track 235.5 -> 0.00 mm, vias 12 -> 0
- net GND: track 230.2 -> 0.00 mm, vias 34 -> 0
- net VCC: track 140.7 -> 0.00 mm, vias 2 -> 0
- net +9V: track 97.7 -> 0.00 mm, vias 1 -> 0
- net GNDA: track 73.9 -> 0.00 mm, vias 13 -> 0
- net /SCL: track 72.2 -> 0.00 mm, vias 1 -> 0
- net /SDA: track 66.9 -> 0.00 mm, vias 1 -> 0
- net Net-(ARDUINO1-Pad19): track 43.3 -> 0.00 mm
- net Net-(C1-Pad1): track 42.2 -> 0.00 mm
- net Net-(D1-Pad4): track 38.4 -> 0.00 mm
- net Net-(ARDUINO1-Pad20): track 37.6 -> 0.00 mm
- net Net-(D1-Pad2): track 37.3 -> 0.00 mm
- net Net-(ARDUINO1-Pad21): track 33.3 -> 0.00 mm
- net Net-(ARDUINO1-Pad22): track 29.0 -> 0.00 mm
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- removed copper zone on B.Cu, net GND
- removed copper zone on F.Cu, net GND
- removed copper zone on B.Cu, net GNDA
- removed copper zone on F.Cu, net GNDA
- removed copper zone on F.Cu, net VCC
Other:
- outline, holes or cut-outs redrawn
- board text removed: "+"
- board text removed: "-"
- board text removed: "0A"
- board text removed: "0B"
- board text removed: "0W"
- board text removed: "1A"
- board text removed: "1B"
- board text removed: "1W"
- board text removed: "2A"
- board text removed: "2B"
- board text removed: "2W"
- board text removed: "3A"
- board text removed: "3B"
- board text removed: "3W"
- board text removed: "4X Digital Potentiometer"
- board text removed: "5.6n"
- board text removed: "9V"
- board text removed: "A"
- board text removed: "A0"
- board text removed: "A1"
- board text removed: "AUX"
- board text removed: "Arduino module for Portable Speaker"
- board text removed: "B"
- board text removed: "C"
- board text removed: "Dat"
- board text removed: "G"
- board text removed: "GND"
- board text removed: "INT"
- board text removed: "Low noise mic preamp"
- board text removed: "MCP4461"
- board text removed: "MIC"
- board text removed: "MISO"
- board text removed: "MOSI"
- board text removed: "NPPC 2019"
- board text removed: "OUT"
- board text removed: "PWR"
- board text removed: "RST"
- board text removed: "S"
- board text removed: "SCK"
- board text removed: "SCL"
- board text removed: "SDA"
- board text removed: "TDA7440 Audio Processor"
- board text removed: "WP"
- board text removed: "nppc 2019"
- board text removed: "preamp"
